Commit message: acc_code_for_magpie
Signed-off-by: Mihir Kulkarni <mihirk284@gmail.com>

File: resources/robots/lmf2/model.urdf (robot description, URDF)
Before this commit: robot quadrotor, 5 links, 4 joints
Links:
- link base_link: geometry collision box size=0.7 0.7 0.5; visual box size=0.4 0.4 0.025
